Commit message: final

File: sim/robot.urdf (robot description, URDF)
Before this commit: robot sentry_lift_test, 13 links, 12 joints
Links:
- link chassis: geometry visual box size=.01 .45 .04; visual box size=.01 .45 .04
- link livox_frame: geometry visual mesh filename=file:///home/dengjiaxi/simulation_seu/navigatiosim2/src/pb2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 scale=1 1 1
Joints:
- joint lift_joint: limit lower=0 upper=.3 effort=300 velocity=.25 -> lower=0 upper=.3 effort=300 velocity=.8
